File: uno-shield/uno-shield-programmer.kicad_pcb (KiCad board)
At the start: 2 copper layers, 57.3 x 53.3 mm, 18 parts, among them J1 Power, J2 Digital/PWM, J3 Analog, J4 Digital/PWM, J5 Conn_01x04_Female, J6 Conn_01x04_Female, U1 ATtiny85-20P

Commit message: move stuff to uno-specific project, add 10uF cap, change to 0603 instead of 0402
Parts:
- added C1: 10u, Capacitor_SMD:C_0603_1608Metric, F.Cu at (134.5, 85.8)
- D1, D2, D3: footprint LED_SMD:LED_0402_1005Metric -> LED_SMD:LED_0603_1608Metric
- moved D3 2.75 mm to (145.8, 72.0)
- moved R3 2.75 mm to (145.8, 76.0)
- moved REF** 2.69 mm to (145.0, 85.5)
- moved D2 0.65 mm to (141.7, 72.0)
- moved R2 0.65 mm to (141.7, 76.0)
- moved D1 0.10 mm to (139.1, 72.0)
- moved R1 0.10 mm to (139.1, 76.0)
- moved J5 0.09 mm to (123.2, 61.0)
Routing:
- net /SCL/A5: track 0.00 -> 90.2 mm, vias 0 -> 1
- net /SDA/A4: track 0.00 -> 87.2 mm, vias 0 -> 2
- net GND: track 119.5 -> 84.1 mm, vias 0 -> 1
- net /~{RESET}: track 0.00 -> 11.9 mm
- net +5V: track 58.6 -> 52.4 mm
- net /7: track 23.4 -> 22.0 mm
- net /8: track 22.6 -> 22.0 mm

Commit message: uno v0.2
Other:
- board text added: "ATtiny Uno Shield v0.2"
- board text removed: "ATtiny Programmer v0.1"
Changed lines of the file:
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@@
     (effects (font (size 1.25 1.25) (thickness 0.2)))
   )
-  (gr_text "ATtiny Programmer v0.1" (at 114 83 90) (layer "F.SilkS")
+  (gr_text "ATtiny Uno Shield v0.2" (at 114 83 90) (layer "F.SilkS")
     (effects (font (size 1.25 1.25) (thickness 0.2)))
   )
